Commit message: fix sim_isaac param not being used

File: urdf/ur.urdf.xacro (robot description, xacro)
@@ -44,4 +44,5 @@
    <xacro:arg name="sim_gazebo" default="false" />
    <xacro:arg name="sim_ignition" default="false" />
+   <xacro:arg name="sim_isaac" default="false" />
    <xacro:arg name="simulation_controllers" default="" />
    <!-- initial position for simulations (Fake Hardware, Gazebo, Ignition) -->
@@ -51,4 +52,5 @@
    <xacro:property name="is_sim_gazebo" value="$(arg sim_gazebo)"/>
    <xacro:property name="is_sim_ignition" value="$(arg sim_ignition)"/>
+   <xacro:property name="is_sim_isaac" value="$(arg sim_isaac)"/>
    <!-- create link fixed to the "world" -->
    <link name="world" />
@@ -94,4 +96,5 @@
      sim_gazebo="$(arg sim_gazebo)"
      sim_ignition="$(arg sim_ignition)"
+     sim_isaac="$(arg sim_isaac)"
      headless_mode="$(arg headless_mode)"
      initial_positions="${xacro.load_yaml(initial_positions_file)}"

File: urdf/ur_macro.xacro (robot description, xacro)
@@ -62,4 +62,5 @@
     sim_gazebo:=false
     sim_ignition:=false
+    sim_isaac:=false
     headless_mode:=false
     initial_positions:=${dict(shoulder_pan_joint=0.0,shoulder_lift_joint=-1.57,elbow_joint=0.0,wrist_1_joint=-1.57,wrist_2_joint=0.0,wrist_3_joint=0.0)}
@@ -103,4 +104,5 @@
         headless_mode="${headless_mode}"
         sim_gazebo="${sim_gazebo}"
+        sim_isaac="${sim_isaac}"
         sim_ignition="${sim_ignition}"
         script_filename="${script_filename}"
