Commit message: move gripper into place

File: urdf/ur5_robotiq85_gripper.urdf.xacro (robot description, xacro)
@@ -46,5 +46,5 @@
   <xacro:include filename="$(find robotiq_description)/urdf/robotiq_2f_85_macro.urdf.xacro" />
   <xacro:robotiq_gripper name="RobotiqGripperHardwareInterface" prefix="" parent="robotiq_coupler" use_fake_hardware="$(arg use_fake_hardware)">
-      <origin xyz="0 0 0.01726" rpy="0 0 0"/>
+      <origin xyz="0 0 0.011" rpy="0 0 0"/>
   </xacro:robotiq_gripper>
   <gazebo reference="wrist_3_joint">

Commit message: update to match isaac sim

File: urdf/ur5_robotiq85_gripper.urdf.xacro (robot description, xacro)
@@ -8,5 +8,8 @@
   <xacro:arg name="name" default="ur"/>
   <xacro:arg name="ur_type" default="ur5"/>
+  <xacro:arg name="sim_isaac" default="false" />
+  <xacro:arg name="use_fake_hardware" default="false" />
   <xacro:include filename="$(find ur_description)/urdf/ur.urdf.xacro" />
+<!--
   <material name="black">
     <color rgba="0 0 0 1"/>
@@ -43,9 +46,10 @@
     <material>Gazebo/FlatBlack</material>
   </gazebo>
-  <xacro:arg name="use_fake_hardware" default="false" />
+  -->
   <xacro:include filename="$(find robotiq_description)/urdf/robotiq_2f_85_macro.urdf.xacro" />
-  <xacro:robotiq_gripper name="RobotiqGripperHardwareInterface" prefix="" parent="robotiq_coupler" use_fake_hardware="$(arg use_fake_hardware)">
-      <origin xyz="0 0 0.011" rpy="0 0 0"/>
+  <xacro:robotiq_gripper name="RobotiqGripperHardwareInterface" prefix="" parent="wrist_3_link" use_fake_hardware="$(arg use_fake_hardware)" sim_isaac="$(arg sim_isaac)">
+      <origin xyz="0 0 0" rpy="0 0 1.5708"/>
   </xacro:robotiq_gripper>
+<!--
   <gazebo reference="wrist_3_joint">
     <provideFeedback>true</provideFeedback>
@@ -59,4 +63,5 @@
     </plugin>
   </gazebo>
+  -->
   <gazebo>
     <gripper name="gazebo_gripper">
